File: outputs/Outputs/Outputs.kicad_sch (KiCad schematic)
At the start: 0 parts

Commit message: Added schematic for nema-17
Parts:
- added A1: Pololu_Breakout_DRV8825, Module:Pololu_Breakout-16_15.2x20.3mm, symbol Driver_Motor:Pololu_Breakout_DRV8825
- added C1: C, symbol Device:C
- added M1: Stepper_Motor_bipolar, symbol Motor:Stepper_Motor_bipolar
Connections:
- new net: A1.3 (A2), M1.1
- new net: A1.4 (A1), M1.2 (-)
- new net: A1.5 (B1), M1.3
- new net: A1.6 (B2), M1.4
- new net +12V: A1.8 (VMOT), C1.1
- new net GND_arduino: A1.1 (GND)
- new net GND_motor: A1.7 (GND), C1.2
- new net VDD_arduino: A1.13 (~{RST}), A1.14 (~{SLP})
- new net arduino_D0: A1.15 (STEP)
- new net arduino_D1: A1.16 (DIR)
Other:
- added sheet nema17_stepper (nema17_stepper.kicad_sch)
