File: power-and-safety/Power-and-Safety/Power-and-Safety.kicad_sch (KiCad schematic)
At the start: 0 parts

Commit message: Added schematic for nema-17
Parts:
- added A2: Arduino_UNO_R2, Module:Arduino_UNO_R2, symbol MCU_Module:Arduino_UNO_R2
Changed lines of the file:
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@@
 	(generator_version "9.0")
 	(paper "A4")
+	(symbol
+		(lib_id "MCU_Module:Arduino_UNO_R2")
+		(at 132.08 101.6 0)
+		(unit 1)
+		(exclude_from_sim no)
+		(in_bom yes)
+		(on_board yes)
+		(dnp no)
+		(fields_autoplaced yes)
+		(property "Reference" "A2"
+			(at 139.3033 73.66 0)
+			(effects
+				(font
+					(size 1.27 1.27)
+				)
+				(justify left)
+			)
+		)
+		(property "Value" "Arduino_UNO_R2"
+			(at 139.3033 76.2 0)
+			(effects
+				(font
+					(size 1.27 1.27)
+				)
+				(justify left)
+			)
+		)
+		(property "Footprint" "Module:Arduino_UNO_R2"
+			(at 132.08 101.6 0)
+			(effects
+				(font
+					(size 1.27 1.27)
+					(italic yes)
+				)
+				(hide yes)
+			)
+		)
+		(property "Datasheet" "https://www.arduino.cc/en/Main/arduinoBoardUno"
+			(at 132.08 101.6 0)
+			(effects
+				(font
+					(size 1.27 1.27)
+				)
+				(hide yes)
+			)
+		)
+		(property "Description" "Arduino UNO Microcontroller Module, release 2"
+			(at 132.08 101.6 0)
+			(effects
+				(font
+					(size 1.27 1.27)
+				)
+				(hide yes)
+			)
+		)
+		(pin "25"
+		)
+		(pin "15"
+		)
+		(pin "21"
+		)
+		(pin "17"
+		)
+		(pin "23"
+		)
+		(pin "6"
+		)
+		(pin "4"
+		)
+		(pin "14"
+		)
+		(pin "11"
+		)
+		(pin "9"
+		)
+		(pin "18"
+		)
+		(pin "2"
+		)
+		(pin "24"
+		)
+		(pin "3"
+		)
+		(pin "16"
+		)
+		(pin "13"
+		)
+		(pin "12"
+		)
+		(pin "26"
+		)
+		(pin "1"
+		)
+		(pin "19"
+		)
+		(pin "28"
+		)
+		(pin "22"
+		)
+		(pin "20"
+		)
+		(pin "29"
+		)
+		(pin "7"
+		)
+		(pin "5"
+		)
+		(pin "27"
+		)
+		(pin "8"
+		)
+		(pin "30"
+		)
+		(pin "10"
+		)
+		(instances
+			(project ""
+				(path "/e28a5393-a52f-43fd-ab49-3e8cb48472a2"
+					(reference "A2")
+					(unit 1)
+				)
+			)
+		)
+	)
+	(symbol
+		(lib_id "power:+7.5V")
+		(at 171.45 59.69 0)
+		(unit 1)
+		(exclude_from_sim no)
+		(in_bom yes)
+		(on_board yes)
+		(dnp no)
+		(fields_autoplaced yes)
+		(property "Reference" "#PWR01"
+			(at 171.45 63.5 0)
+			(effects
+				(font
+					(size 1.27 1.27)
+				)
+				(hide yes)
+			)
+		)
+		(property "Value" "+7.4V"
+			(at 171.45 54.61 0)
+			(effects
+				(font
+					(size 1.27 1.27)
+				)
+			)
+		)
+		(property "Footprint" ""
+			(at 171.45 59.69 0)
+			(effects
+				(font
+					(size 1.27 1.27)
+				)
+				(hide yes)
+			)
+		)
+		(property "Datasheet" ""
+			(at 171.45 59.69 0)
+			(effects
+				(font
+					(size 1.27 1.27)
+				)
+				(hide yes)
+			)
+		)
+		(property "Description" "Power symbol creates a global label with name \"+7.5V\""
+			(at 171.45 59.69 0)
+			(effects
+				(font
+					(size 1.27 1.27)
+				)
+				(hide yes)
+			)
+		)
+		(pin "1"
+		)
+		(instances
+			(project ""
+				(path "/e28a5393-a52f-43fd-ab49-3e8cb48472a2"
+					(reference "#PWR01")
+					(unit 1)
+				)
+			)
+		)
+	)
 	(sheet_instances
 		(path "/"
