File: power-and-safety/Power-and-Safety/Power-and-Safety.kicad_sch (KiCad schematic)
At the start: 0 parts

Commit message: Added emergency turn off circuit for Microcontroller.
Parts:
- added D1: 1N4148WT, Diode_SMD:D_SOD-523, symbol Diode:1N4148WT
- added Q1: NMOS, symbol Simulation_SPICE:NMOS
- added R1, R2, R3, R4, R5, R6: R, symbol Device:R
- added SW1: SW_Push, symbol Switch:SW_Push
Connections:
- new net: Q1.1 (D), R4.2
- new net: Q1.3 (S), R5.1, R6.1
- new net: D1.1 (K), Q1.2 (G), SW1.1
- new net: R3.2, SW1.2
- new net +12V: R1.1, R3.1, R4.1
- new net Arduino_A0: R1.2, R2.1
- new net Arduino_D0: D1.2 (A)
- new net Arduino_VIN: R5.2
- new net GND: R2.2
- new net Motors: R6.2

Commit message: added textbox note.
Parts:
- removed R4: R, symbol Device:R
Connections:
- net +12V: now also Q1.1 (D)
Changed lines of the file:
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@@
-	(wire
-		(pts
-			(xy 187.96 59.69) (xy 187.96 62.23)
-		)
-		(stroke
-			(width 0)
-			(type default)
-		)
-	)
 	(wire
 		(pts
@@
 	(wire
 		(pts
-			(xy 187.96 69.85) (xy 187.96 92.71)
-		)
-		(stroke
-			(width 0)
-			(type default)
-		)
-	)
-	(wire
-		(pts
 			(xy 175.26 69.85) (xy 175.26 80.01)
 		)
@@
 		(pts
 			(xy 172.72 107.95) (xy 187.96 107.95)
+		)
+		(stroke
+			(width 0)
+			(type default)
+		)
+	)
+	(wire
+		(pts
+			(xy 187.96 59.69) (xy 187.96 92.71)
 		)
 		(stroke
@@
 		)
 	)
-	(symbol
-		(lib_id "Device:R")
-		(at 187.96 66.04 0)
-		(unit 1)
-		(exclude_from_sim no)
-		(in_bom yes)
-		(on_board yes)
-		(dnp no)
-		(fields_autoplaced yes)
-		(property "Reference" "R4"
-			(at 190.5 64.7699 0)
-			(effects
-				(font
-					(size 1.27 1.27)
-				)
-				(justify left)
-			)
-		)
-		(property "Value" "R"
-			(at 190.5 67.3099 0)
-			(effects
-				(font
-					(size 1.27 1.27)
-				)
-				(justify left)
-			)
-		)
-		(property "Footprint" ""
-			(at 186.182 66.04 90)
-			(effects
-				(font
-					(size 1.27 1.27)
-				)
-				(hide yes)
-			)
-		)
-		(property "Datasheet" "~"
-			(at 187.96 66.04 0)
-			(effects
-				(font
-					(size 1.27 1.27)
-				)
-				(hide yes)
-			)
-		)
-		(property "Description" "Resistor"
-			(at 187.96 66.04 0)
-			(effects
-				(font
-					(size 1.27 1.27)
-				)
-				(hide yes)
-			)
-		)
-		(pin "2"
-		)
-		(pin "1"
-		)
-		(instances
-			(project "Power-and-Safety"
-				(path "/e28a5393-a52f-43fd-ab49-3e8cb48472a2"
-					(reference "R4")
-					(unit 1)
-				)
-			)
-		)
-	)

Commit message: edited voltage splits.
Parts:
- removed D1: 1N4148WT, Diode_SMD:D_SOD-523, symbol Diode:1N4148WT
- removed Q1: NMOS, symbol Simulation_SPICE:NMOS
- removed R1, R2, R3, R5, R6: R, symbol Device:R
- removed SW1: SW_Push, symbol Switch:SW_Push
Other:
- added sheet voltage_splits (voltage_splits.kicad_sch)

Commit message: worked on emergency power shutoff
Other:
- added sheet emergency_shutoff (emergency_shutoff.kicad_sch)
Changed lines of the file:
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@@
 	(paper "A4")
+	(sheet
+		(at 631.825 1.27)
+		(size 302.895 205.74)
+		(exclude_from_sim no)
+		(in_bom yes)
+		(on_board yes)
+		(dnp no)
+		(fields_autoplaced yes)
+		(stroke
+			(width 0.1524)
+			(type solid)
+		)
+		(fill
+			(color 0 0 0 0.0000)
+		)
+		(property "Sheetname" "emergency_shutoff"
+			(at 631.825 0.5584 0)
+			(effects
+				(font
+					(size 1.27 1.27)
+				)
+				(justify left bottom)
+			)
+		)
+		(property "Sheetfile" "emergency_shutoff.kicad_sch"
+			(at 631.825 207.5946 0)
+			(effects
+				(font
+					(size 1.27 1.27)
+				)
+				(justify left top)
+			)
+		)
+		(instances
+			(project "Power-and-Safety"
+				(path "/e28a5393-a52f-43fd-ab49-3e8cb48472a2"
+					(page "3")
+				)
+			)
+		)
+	)
 	(sheet
 		(at 323.85 1.27)
