File: power-and-safety/Power-and-Safety/voltage_splits.kicad_sch (KiCad schematic)
At the start: 3 parts

Commit message: worked on emergency power shutoff
Connections:
- net +12V renamed 12V_motor
Changed lines of the file:
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@@
 			)
 		)
-		(property "Value" "+12V"
-			(at 123.19 22.86 0)
-			(effects
-				(font
-					(size 1.27 1.27)
-				)
+		(property "Value" "12V_motor"
+			(at 125.73 26.6699 0)
+			(effects
+				(font
+					(size 1.27 1.27)
+				)
+				(justify left)
 			)
 		)
@@
 				)
 			)
+			(project "Power-and-Safety"
+				(path "/e28a5393-a52f-43fd-ab49-3e8cb48472a2/d36d0e8d-00a1-4cf6-8b6f-69f787e31cd0"
+					(reference "#PWR?")
+					(unit 1)
+				)
+			)
 		)
 	)
@@
 					(unit 1)
 				)
+			)
+			(project "Power-and-Safety"
+				(path "/e28a5393-a52f-43fd-ab49-3e8cb48472a2/d36d0e8d-00a1-4cf6-8b6f-69f787e31cd0"
+					(reference "#PWR?")
+					(unit 1)
+				)
